Commit message: Can simulate roughly with teb.

File: nav2_run/urdf/diff_drive.urdf (robot description, URDF)
Before this commit: robot sam_bot, 3 links, 2 joints
Joints:
- joint caster_joint: axis (none) -> 0 1 0; type fixed -> continuous

Commit message: Lidar is ok.

File: nav2_run/urdf/diff_drive.urdf (robot description, URDF)
Before this commit: robot sam_bot, 3 links, 2 joints
Links:
- added link imu_link; collision box size=0.1 0.1 0.1; visual box size=0.1 0.1 0.1
- added link lidar_link; collision cylinder length=0.18 radius=0.0508; visual cylinder length=0.18 radius=0.0508
Joints:
- added joint imu_joint: type fixed, parent base_link, child imu_link, origin xyz=0 0 0.01
- added joint lidar_joint: type fixed, parent base_link, child lidar_link, origin xyz=0.0 0.0 ${base_height/2 + 0.18/2} rpy=0 0 0

Commit message: Modify the car module to be more real.

File: nav2_run/urdf/diff_drive.urdf (robot description, URDF)
Before this commit: robot sam_bot, 5 links, 4 joints
Links:
- link front_caster: geometry collision sphere radius=${wheel_radius-wheel_zoff}; visual sphere radius=${wheel_radius-wheel_zoff}

Commit message: Change to 2 caster in model.

File: nav2_run/urdf/diff_drive.urdf (robot description, URDF)
Before this commit: robot sam_bot, 5 links, 4 joints
Links:
- removed link front_caster
- link lidar_link: geometry collision cylinder length=0.09 radius=0.0508; visual cylinder length=0.09 radius=0.0508
Joints:
- removed joint caster_joint
- joint lidar_joint: origin xyz=0.0 0.0 ${base_height/2 + 0.18/2} rpy=0 0 0 -> xyz=0.0 0.0 ${base_height/2 + 0.09/2} rpy=0 0 0
